File: pcb/jardim.sch (EAGLE design)
At the start: 9 parts, among them U2 7805

Commit message: pcb: LEDs
Parts:
- added C5, C6: 22pF, SparkFun-Capacitors:CAPKIT
- added C7: CAP-09538, SparkFun-Capacitors:1000UF-25V(PTH)
- added D3, D5: (no value), SparkFun-LED:LED3MM
- added D4: 1N4001, SparkFun-DiscreteSemi:DIODEKIT2
- added IC1, IC2, IC3: 74LS595N, SparkFun-DigitalIC:74LS595N
- added J2: Power Select, SparkFun-Connectors:M03PTH
- added J3: USB to Serial, SparkFun-Connectors:M06SILK_FEMALE_PTH
- added J4: C485, SparkFun-Connectors:M025MM
- added J5: Power LED, SparkFun-Connectors:M025MM
- added J6: Mode Select, SparkFun-Connectors:M03PTH
- added R10, R11, R12, R13, R14, R15, R16, R17, R18, R19, R20, R21, R22, R23, R24, R25, R26, R27, R4, R5, R6, R7, R8, R9: (no value), resistor-power:RCA4080
- added R2: 470R, SparkFun-Resistors:RESISTORPTH-1/4W
- added R28: 1k, SparkFun-Resistors:RESISTORPTH-1/4W
- added R3: 10k, SparkFun-Resistors:RESISTORPTH-1/4W
- added S1: SWITCH-MOMENTARY-2PTH, SparkFun-Electromechanical:SWITCH-MOMENTARY-2PTH
- added U$1: MAX485DIL, SparkFun-DigitalIC:MAX485DIL
- added U1: ATMEGA328P_PDIP, SparkFun-DigitalIC:ATMEGA328P_PDIP
- added ULN1, ULN2, ULN3: (no value), SparkFun-PowerIC:ULN2803DIP
- added X1, X2, X3, X4, X5, X6, X7, X8: (no value), con-wago-500:W237-4
- added Y1: 16MHz, SparkFun-FreqCtrl:CRYSTALHC49US
- J1: value (none) -> Power In
Connections:
- removed net 5V: C3.+, C4.1, R1.2, U2.OUT
- new net ARDUINO_D10: IC1.RCK, IC2.RCK, IC3.RCK, U1.PB2(SS/OC1B)
- new net ARDUINO_D11: IC1.SER, U1.PB3(MOSI/OC2)
- new net ARDUINO_D12: J6.2, U1.PB4(MISO)
- new net ARDUINO_D13: IC1.SCK, IC2.SCK, IC3.SCK, U1.PB5(SCK)
- new net ARDUINO_D3: R2.2, U1.PD3(INT1)
- new net FTDI_CTS: J3.5
- new net FTDI_DTR: J3.1, R3.1, S1.1, U1.PC6(/RESET)
- new net FTDI_RX: J3.2, U$1.DI, U1.PD1(TXD)
- new net FTDI_TX: J3.3, U$1.RO, U1.PD0(RXD)
- new net FTDI_VCC: J2.1, J3.4
- new net N$1: R4.1, ULN1.18
- new net N$10: U$1.DE, U$1.RE
- new net N$11: J4.1, U$1.A
- new net N$12: J4.2, U$1.B
- new net N$13: R6.1, ULN1.16
- new net N$14: R7.2, X2-2.KL
- new net N$15: R7.1, ULN1.15
- new net N$16: R8.1, ULN1.14
- new net N$17: R9.1, ULN1.13
- new net N$18: R4.2, X1-2.KL
- new net N$19: R5.2, X1-3.KL
- new net N$20: R6.2, X1-4.KL
- new net N$21: R10.1, ULN1.12
- new net N$22: IC1.QA, ULN1.1
- new net N$23: IC1.QB, ULN1.2
- new net N$24: IC1.QC, ULN1.3
- new net N$25: IC1.QD, ULN1.4
- new net N$26: IC1.QE, ULN1.5
- new net N$27: IC1.QF, ULN1.6
- new net N$28: IC1.QG, ULN1.7
- new net N$29: IC1.QH, ULN1.8
- new net N$30: R8.2, X2-3.KL
- new net N$31: R9.2, X2-4.KL
- new net N$32: R11.1, ULN1.11
- new net N$33: R12.1, ULN2.18
- new net N$34: R13.1, ULN2.17
- new net N$35: R14.1, ULN2.16
- new net N$36: R10.2, X3-2.KL
- new net N$37: R11.2, X3-3.KL
- new net N$38: R12.2, X3-4.KL
- new net N$39: R15.1, ULN2.15
- new net N$4: C5.2, U1.PB6(XTAL1/TOSC1), Y1.1
- new net N$40: R16.1, ULN2.14
- new net N$41: R17.1, ULN2.13
- new net N$42: R18.1, ULN2.12
- new net N$43: R13.2, X4-2.KL
- new net N$44: R14.2, X4-3.KL
- new net N$45: R15.2, X4-4.KL
- new net N$46: R19.1, ULN2.11
- new net N$47: IC2.QA, ULN2.1
- new net N$48: R20.1, ULN3.18
- new net N$49: R21.1, ULN3.17
- new net N$5: C6.1, U1.PB7(XTAL2/TOSC2), Y1.2
- new net N$50: R16.2, X5-2.KL
- new net N$51: R17.2, X5-3.KL
- new net N$52: R18.2, X5-4.KL
- new net N$53: R22.1, ULN3.16
- new net N$54: R23.1, ULN3.15
- new net N$55: R24.1, ULN3.14
- new net N$56: R25.1, ULN3.13
- new net N$57: R19.2, X6-2.KL
- new net N$58: R20.2, X6-3.KL
- new net N$59: R21.2, X6-4.KL
- new net N$6: D3.A, R2.1
- new net N$60: R26.1, ULN3.12
- new net N$61: R27.1, ULN3.11
- new net N$62: IC2.QB, ULN2.2
- new net N$63: IC2.QC, ULN2.3
- new net N$64: R22.2, X7-2.KL
- new net N$65: R23.2, X7-3.KL
- new net N$66: R24.2, X7-4.KL
- new net N$67: IC2.QD, ULN2.4
- new net N$68: IC2.QE, ULN2.5
- new net N$69: IC2.QF, ULN2.6
- new net N$7: D4.A, J5.2
- new net N$70: IC2.QG, ULN2.7
- new net N$71: R25.2, X8-2.KL
- new net N$72: R26.2, X8-3.KL
- new net N$73: R27.2, X8-4.KL
- new net N$74: C7.+, D4.C, R28.2, ULN1.10, ULN2.10, ULN3.10
- new net N$75: IC2.QH, ULN2.8
- new net N$76: IC3.QA, ULN3.1
- new net N$77: IC3.QB, ULN3.2
- new net N$78: IC3.QC, ULN3.3
- new net N$79: IC3.QD, ULN3.4
- new net N$80: IC3.QE, ULN3.5
- new net N$81: IC3.QF, ULN3.6
- new net N$82: IC3.QG, ULN3.7
- new net N$83: IC3.QH, ULN3.8
- new net N$84: D5.A, R28.1
- new net N$85: J2.3, U2.OUT
- new net N$87: IC1.QH*, IC2.SER
- new net N$88: IC2.QH*, IC3.SER
- new net N$9: R5.1, ULN1.17
- new net VCC: C3.+, C4.1, IC1.SCL, IC1.VCC, IC2.SCL, IC2.VCC, IC3.SCL, IC3.VCC, J2.2, J6.1, R1.2, R3.2, U$1.VCC, U1.AREF, U1.AVCC, U1.VCC
- net GND: now also C5.1, C6.2, C7.-, D3.C, D5.C, IC1.G, IC1.GND, IC2.G, IC2.GND, IC3.G, IC3.GND, J3.6, J5.1, J6.3, S1.2, U$1.GND, U1.GND@1, U1.GND@2, ULN1.9, ULN2.9, ULN3.9
Other:
- moved on the sheet: C1, C2, C3, C4, D1, D2, J1, R1, U2

Commit message: pcb: 1N4001 -> 1N4007
Parts:
- D4: value 1N4001 -> 1N4007; device SparkFun-DiscreteSemi:DIODEKIT2 -> SparkFun-DiscreteSemi:DIODEPTH
Changed lines of the file:
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@@
 <part name="GND12" library="SparkFun-Aesthetics" deviceset="GND" device=""/>
 <part name="C7" library="SparkFun-Capacitors" deviceset="1000UF-25V(PTH)" device="" value="CAP-09538"/>
-<part name="D4" library="SparkFun-DiscreteSemi" deviceset="DIODE" device="KIT2" value="1N4001"/>
 <part name="R28" library="SparkFun-Resistors" deviceset="RESISTOR" device="PTH-1/4W" value="1k"/>
 <part name="D5" library="SparkFun-LED" deviceset="LED" device="3MM"/>
 <part name="SUPPLY11" library="SparkFun-Aesthetics" deviceset="VCC" device=""/>
 <part name="GND13" library="SparkFun-Aesthetics" deviceset="GND" device=""/>
+<part name="D4" library="SparkFun-DiscreteSemi" deviceset="DIODE" device="PTH" value="1N4007"/>
 </parts>
 <sheets>
@@
 <instance part="GND12" gate="1" x="281.94" y="-7.62"/>
 <instance part="C7" gate="G$1" x="480.06" y="60.96"/>
-<instance part="D4" gate="G$1" x="472.44" y="78.74" rot="R270"/>
 <instance part="R28" gate="G$1" x="492.76" y="66.04" rot="R180"/>
 <instance part="D5" gate="G$1" x="500.38" y="60.96"/>
 <instance part="SUPPLY11" gate="G$1" x="53.34" y="20.32" rot="MR0"/>
 <instance part="GND13" gate="1" x="53.34" y="-12.7" rot="MR0"/>
+<instance part="D4" gate="G$1" x="472.44" y="78.74" rot="R270"/>
 </instances>
 <busses>
@@
 <pinref part="C7" gate="G$1" pin="+"/>
 <wire x1="480.06" y1="66.04" x2="480.06" y2="63.5" width="0.1524" layer="91"/>
-<pinref part="D4" gate="G$1" pin="C"/>
 <wire x1="472.44" y1="76.2" x2="472.44" y2="66.04" width="0.1524" layer="91"/>
 <pinref part="R28" gate="G$1" pin="2"/>
 <wire x1="487.68" y1="66.04" x2="480.06" y2="66.04" width="0.1524" layer="91"/>
 <junction x="480.06" y="66.04"/>
+<pinref part="D4" gate="G$1" pin="C"/>
 </segment>
 </net>
@@
 <segment>
 <pinref part="J5" gate="G$1" pin="2"/>
+<wire x1="472.44" y1="83.82" x2="472.44" y2="81.28" width="0.1524" layer="91"/>
 <pinref part="D4" gate="G$1" pin="A"/>
-<wire x1="472.44" y1="83.82" x2="472.44" y2="81.28" width="0.1524" layer="91"/>
-</segment>
-</net>
+</segment>
+</net>
